File: pcb/LVDS Raspi V0.brd (EAGLE design)
At the start: 45 x 67 mm, 26 parts

Commit message: rounder lines are better lines
Parts:
- R1, R2, R3, R4, R5, R6, R7, R8: value (none) -> 0
Connections:
- net +3V3: now also FIX-30P-D6.3
- net GND: now also FIX-30P-D6.25, FIX-30P-D6.26
Routing:
- net +3V3: track 141.2 -> 144.0 mm
- net GND: vias 2 -> 5
Other:
- board size 45 x 67 mm -> 41 x 67 mm
- board text added: "LVDS-Shield 1.0 Philip Caroli"
